Commit message: added camera

File: models/basic_mobile_bot_v2.urdf (robot description, URDF)
Before this commit: robot basic_mobile_bot, 6 links, 5 joints
Links:
- added link camera_depth_frame
- added link camera_link, mass 0.035; collision box size=0.015 0.130 0.022; visual box size=0.015 0.130 0.022
Joints:
- added joint camera_depth_joint: type fixed, parent camera_link, child camera_depth_frame, origin xyz=0 0 0 rpy=${-pi/2} 0 ${-pi/2}
- added joint camera_joint: type fixed, parent base_link, child camera_link, origin xyz=0.35 0 0.05 rpy=0 0 0
